File: PCB/trhw.kicad_sch (KiCad schematic)
At the start: 46 parts, among them J1 USB_C_Receptacle_USB2.0_14P, J2 Conn_01x02, J3 Conn_01x15, J4 Conn_01x16, SW1 SW_Push, U1 RP2040, U2 W25Q32JVSS, U3 TPS63001, U4 Raspberry Pi Radio Module 2, U5 TP4056-42-ESOP8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

Commit message: Final
Parts:
- added C19, C20, C21, C22: 100n, Capacitor_SMD:C_0402_1005Metric, symbol Device:C
- added D4, D5, D6, D7: WS2812B, LED_SMD:LED_WS2812B_PLCC4_5.0x5.0mm_P3.2mm, symbol LED:WS2812B
- added SW2, SW3, SW4, SW5: SW_Push, Button_Switch_SMD:SW_SPST_B3U-1000P, symbol Switch:SW_Push
Connections:
- net +3V3: now also C19.1, C20.1, C21.1, C22.1, D4.1 (VDD), D5.1 (VDD), D6.1 (VDD), D7.1 (VDD)
- net GND: now also C19.2, C20.2, C21.2, C22.2, D4.3 (VSS), D5.3 (VSS), D6.3 (VSS), D7.3 (VSS), SW2.2, SW3.2, SW4.2, SW5.1
- net GP4: now also D4.4 (DIN)
- net GP5: now also SW2.1
- net GP6: now also SW3.1
- net GP7: now also SW4.1
- net VCC: now reaches C15.1, D1.1 (K), D2.1 (K), R3.1, U3.5 (VIN)
- net at U1.26 (RUN): now also SW5.2
- new net: D5.2 (DOUT), D6.4 (DIN)
- new net: D4.2 (DOUT), D5.4 (DIN)
- new net: D6.2 (DOUT), D7.4 (DIN)
- no-connect marks 7 -> 8
